File: shadystake.kicad_sch (KiCad schematic)
At the start: 19 parts, among them J1 6P6C, J2 6P6C, J3 6P6C, J4 6P6C, J5 6P6C, J6 6P6C, J7 8P8C

Commit message: update footprints to have less silkscreening
Parts:
- J1, J2, J3, J4, J5, J6: footprint Connector_RJ:RJ12_Amphenol_54601 -> Shadystake:RJ12_Amphenol_54601
- J7: footprint Connector_RJ:RJ45_Amphenol_54602-x08_Horizontal -> Shadystake:RJ45_Amphenol_54602-x08_Horizontal
Changed lines of the file:
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@@
       (effects (font (size 1.27 1.27)) (justify right))
     )
-    (property "Footprint" "Connector_RJ:RJ45_Amphenol_54602-x08_Horizontal" (id 2) (at 251.46 89.535 90)
+    (property "Footprint" "Shadystake:RJ45_Amphenol_54602-x08_Horizontal" (id 2) (at 251.46 89.535 90)
       (effects (font (size 1.27 1.27)) hide)
     )
@@
     (property "Reference" "J1" (id 0) (at 56.0578 44.0182 0))
     (property "Value" "6P6C" (id 1) (at 56.0578 46.3296 0))
-    (property "Footprint" "Connector_RJ:RJ12_Amphenol_54601" (id 2) (at 54.61 57.785 90)
+    (property "Footprint" "Shadystake:RJ12_Amphenol_54601" (id 2) (at 54.61 57.785 90)
       (effects (font (size 1.27 1.27)) hide)
     )
@@
     (property "Reference" "J2" (id 0) (at 56.0578 69.4182 0))
     (property "Value" "6P6C" (id 1) (at 56.0578 71.7296 0))
-    (property "Footprint" "Connector_RJ:RJ12_Amphenol_54601" (id 2) (at 54.61 83.185 90)
+    (property "Footprint" "Shadystake:RJ12_Amphenol_54601" (id 2) (at 54.61 83.185 90)
       (effects (font (size 1.27 1.27)) hide)
     )
@@
     (property "Reference" "J3" (id 0) (at 56.0578 94.8182 0))
     (property "Value" "6P6C" (id 1) (at 56.0578 97.1296 0))
-    (property "Footprint" "Connector_RJ:RJ12_Amphenol_54601" (id 2) (at 54.61 108.585 90)
+    (property "Footprint" "Shadystake:RJ12_Amphenol_54601" (id 2) (at 54.61 108.585 90)
       (effects (font (size 1.27 1.27)) hide)
     )
@@
     (property "Reference" "J4" (id 0) (at 56.0578 120.2182 0))
     (property "Value" "6P6C" (id 1) (at 56.0578 122.5296 0))
-    (property "Footprint" "Connector_RJ:RJ12_Amphenol_54601" (id 2) (at 54.61 133.985 90)
+    (property "Footprint" "Shadystake:RJ12_Amphenol_54601" (id 2) (at 54.61 133.985 90)
       (effects (font (size 1.27 1.27)) hide)
     )
@@
     (property "Reference" "J6" (id 0) (at 94.1578 107.5182 0))
     (property "Value" "6P6C" (id 1) (at 94.1578 109.8296 0))
-    (property "Footprint" "Connector_RJ:RJ12_Amphenol_54601" (id 2) (at 92.71 121.285 90)
+    (property "Footprint" "Shadystake:RJ12_Amphenol_54601" (id 2) (at 92.71 121.285 90)
       (effects (font (size 1.27 1.27)) hide)
     )
@@
     (property "Reference" "J5" (id 0) (at 94.1578 55.4482 0))
     (property "Value" "6P6C" (id 1) (at 94.1578 57.7596 0))
-    (property "Footprint" "Connector_RJ:RJ12_Amphenol_54601" (id 2) (at 92.71 69.215 90)
+    (property "Footprint" "Shadystake:RJ12_Amphenol_54601" (id 2) (at 92.71 69.215 90)
       (effects (font (size 1.27 1.27)) hide)
     )
@@
     )
     (path "/00000000-0000-0000-0000-00005e77093f"
-      (reference "J1") (unit 1) (value "6P6C") (footprint "Connector_RJ:RJ12_Amphenol_54601")
+      (reference "J1") (unit 1) (value "6P6C") (footprint "Shadystake:RJ12_Amphenol_54601")
     )
     (path "/00000000-0000-0000-0000-00005e774911"
-      (reference "J2") (unit 1) (value "6P6C") (footprint "Connector_RJ:RJ12_Amphenol_54601")
+      (reference "J2") (unit 1) (value "6P6C") (footprint "Shadystake:RJ12_Amphenol_54601")
     )
     (path "/00000000-0000-0000-0000-00005e775c26"
-      (reference "J3") (unit 1) (value "6P6C") (footprint "Connector_RJ:RJ12_Amphenol_54601")
+      (reference "J3") (unit 1) (value "6P6C") (footprint "Shadystake:RJ12_Amphenol_54601")
     )
     (path "/00000000-0000-0000-0000-00005e776296"
-      (reference "J4") (unit 1) (value "6P6C") (footprint "Connector_RJ:RJ12_Amphenol_54601")
+      (reference "J4") (unit 1) (value "6P6C") (footprint "Shadystake:RJ12_Amphenol_54601")
     )
     (path "/7cba2845-987e-4ef7-9f17-6058946e05f1"
-      (reference "J5") (unit 1) (value "6P6C") (footprint "Connector_RJ:RJ12_Amphenol_54601")
+      (reference "J5") (unit 1) (value "6P6C") (footprint "Shadystake:RJ12_Amphenol_54601")
     )
     (path "/723fb613-a350-4201-8db7-5e55947d06e9"
-      (reference "J6") (unit 1) (value "6P6C") (footprint "Connector_RJ:RJ12_Amphenol_54601")
+      (reference "J6") (unit 1) (value "6P6C") (footprint "Shadystake:RJ12_Amphenol_54601")
     )
     (path "/00000000-0000-0000-0000-00005e76be8e"
-      (reference "J7") (unit 1) (value "8P8C") (footprint "Connector_RJ:RJ45_Amphenol_54602-x08_Horizontal")
-    )
-  )
+      (reference "J7") (unit 1) (value "8P8C") (footprint "Shadystake:RJ45_Amphenol_54602-x08_Horizontal")
+    )
+  )
